Commit message: moveit2 integration

File: src/patrick_main/urdf/patrick.urdf.xacro (robot description, xacro)
@@ -119,4 +119,20 @@
   <!-- ================================================================= -->
   <!--  5. ros2_control hardware interface                               -->
+  <!--                                                                   -->
+  <!--  Arm joints use POSITION command interface (works for both        -->
+  <!--  Dynamixel protocol 1 and stepper-with-encoder backends, and is   -->
+  <!--  what joint_trajectory_controller / scaled_joint_trajectory_      -->
+  <!--  controller drive with MoveIt trajectories).                      -->
+  <!--                                                                   -->
+  <!--  Joint5L is declared as a mimic of Joint5R (parallel-jaw gripper) -->
+  <!--  so it has NO command interface exported. In Gazebo Harmonic,     -->
+  <!--  gz_ros2_control honours URDF <mimic> via the ros2_control Mimic  -->
+  <!--  component. On real hardware, ArduinoHardwareInterface replicates -->
+  <!--  the Joint5R command internally.                                  -->
+  <!--                                                                   -->
+  <!--  A GPIO "speed_scaling" is exported so ScaledJointTrajectory-     -->
+  <!--  Controller can slow trajectory execution when the real hardware  -->
+  <!--  reports reduced capability (Dynamixel overload, stall, etc.).    -->
+  <!--  In simulation it is hardcoded to 1.0 by gz_ros2_control.         -->
   <!-- ================================================================= -->
   <ros2_control name="patrick_ros2_control" type="system">
@@ -144,7 +160,7 @@
       <state_interface name="velocity"/>
     </joint>
-    <!-- Arm joints (all via Arduino on real HW) -->
+    <!-- Arm joints (Joint1..Joint4) — position-commanded -->
     <joint name="Joint1">
-      <command_interface name="effort"/>
+      <command_interface name="position"/>
       <state_interface name="position"/>
       <state_interface name="velocity"/>
@@ -152,5 +168,5 @@
     </joint>
     <joint name="Joint2">
-      <command_interface name="effort"/>
+      <command_interface name="position"/>
       <state_interface name="position"/>
       <state_interface name="velocity"/>
@@ -158,5 +174,5 @@
     </joint>
     <joint name="Joint3">
-      <command_interface name="effort"/>
+      <command_interface name="position"/>
       <state_interface name="position"/>
       <state_interface name="velocity"/>
@@ -164,21 +180,30 @@
     </joint>
     <joint name="Joint4">
-      <command_interface name="effort"/>
-      <state_interface name="position"/>
-      <state_interface name="velocity"/>
-      <state_interface name="effort"/>
-    </joint>
+      <command_interface name="position"/>
+      <state_interface name="position"/>
+      <state_interface name="velocity"/>
+      <state_interface name="effort"/>
+    </joint>
+    <!-- Gripper driver joint (Joint5R) — position-commanded -->
     <joint name="Joint5R">
-      <command_interface name="effort"/>
-      <state_interface name="position"/>
-      <state_interface name="velocity"/>
-      <state_interface name="effort"/>
-    </joint>
+      <command_interface name="position"/>
+      <state_interface name="position"/>
+      <state_interface name="velocity"/>
+      <state_interface name="effort"/>
+    </joint>
+    <!-- Gripper mimic joint (Joint5L) — no command interface, mirrors Joint5R
+         with multiplier -1.0 so the jaws move in OPPOSITE directions
+         (parallel-jaw open/close), not together. -->
     <joint name="Joint5L">
-      <command_interface name="effort"/>
-      <state_interface name="position"/>
-      <state_interface name="velocity"/>
-      <state_interface name="effort"/>
-    </joint>
+      <param name="mimic">Joint5R</param>
+      <param name="multiplier">-1.0</param>
+      <state_interface name="position"/>
+      <state_interface name="velocity"/>
+      <state_interface name="effort"/>
+    </joint>
+    <!-- Speed-scaling GPIO (consumed by ur_controllers/ScaledJointTrajectoryController) -->
+    <gpio name="speed_scaling">
+      <state_interface name="speed_scaling_factor"/>
+    </gpio>
   </ros2_control>
   <!-- ================================================================= -->

File: src/patrick_main/urdf/patrick_arm.urdf.xacro (robot description, xacro)
@@ -186,4 +186,9 @@
       <dynamics damping="0.05" friction="0.01"/>
       <limit lower="-0.393" upper="0.393" effort="50" velocity="2"/>
+      <!-- Gripper is a 1-DOF parallel jaw; left finger mirrors right finger.
+           Both joints share the same axis orientation in Link5, so the mimic
+           multiplier must be -1.0 for the fingers to move in OPPOSITE
+           directions (open/close) instead of swaying together. -->
+      <mimic joint="Joint5R" multiplier="-1.0" offset="0.0"/>
     </joint>
     <!-- End-Effector target cube (visual reference) -->
@@ -205,4 +210,15 @@
       <parent link="Link6R"/><child link="target_cube_ee"/>
     </joint>
+    <!-- Tool Center Point (TCP) — virtual frame MoveIt uses as the IK tip.
+         Fixed to Link5 (the wrist, AFTER Joint4 but BEFORE Joint5R/L) so the
+         arm kinematic chain base_link → arm_tool0 only includes Joint1..4
+         (gripper joints stay out of the arm group). Its offset in Link5
+         equals target_cube_ee's world position at Joint5R=0, putting the
+         interactive goal marker between the gripper jaws. -->
+    <link name="arm_tool0"/>
+    <joint name="arm_tool0_joint" type="fixed">
+      <origin xyz="0 0 0.22" rpy="0 0 0"/>
+      <parent link="Link5"/><child link="arm_tool0"/>
+    </joint>
   </xacro:macro>
 </robot>
